File: PCB/power.kicad_sch (KiCad schematic)
At the start: 28 parts, among them Q1 Q_PMOS_SDG, U1 TP4056, U2 HT77xxBA, U3 LM1117-3.3, U4 OP07

Commit message: some updated changes to power circuit
Parts:
- removed C3: 10u, symbol Device:C_Small
- removed C4, C7: 22u, symbol Device:C_Small
- removed C5: 0.1u, symbol Device:C_Small
- removed C6: 47u, symbol Device:C_Small
- removed D1: 1N5819, symbol Device:D_Schottky
- removed D2: 1N5819, Diode_THT:D_DO-41_SOD81_P10.16mm_Horizontal, symbol Diode:1N5817
- removed L1: 47u, symbol Device:L_Small
- removed Q1: Q_PMOS_SDG, symbol Device:Q_PMOS_SDG
- removed R10, R4, R5, R6: 10k, symbol Device:R_Small
- removed R7, R8, R9: 1k, symbol Device:R_Small
- removed U2: HT77xxBA, Package_TO_SOT_SMD:SOT-23-5, symbol Regulator_Switching:AP3012
- removed U3: LM1117-3.3, symbol Regulator_Linear:LM1117-3.3
- removed U4: OP07, symbol Amplifier_Operational:OP07
- added U2: LM2937xMP, Package_TO_SOT_SMD:SOT-223-3_TabPin2, symbol Regulator_Linear:LM2937xMP
- gave numbers to parts that had none: 1
Connections:
- net 3V3: now also U2.3 (VO)
- net GND: now also U2.2 (GND)
- net V_BAT+: now also U2.1 (VI)
Other:
- note removed: "Section C: Booster"
- note removed: "Section D: Polarity Protection and UVLO"
- moved on the sheet: BT1
