File: PCB/Power_Module.kicad_sch (KiCad schematic)
At the start: 10 parts, among them U1 TP4056, U2 LM2937xMP

Commit message: MERGING SCHEMATICS
Parts:
- removed U2: LM2937xMP, Package_TO_SOT_SMD:SOT-223-3_TabPin2, symbol Regulator_Linear:LM2937xMP
- added C3: 10u, symbol Device:C_Small
- added C4: 22u, symbol Device:C_Small
- added C5: 0.1u, symbol Device:C_Small
- added D1, D2: D_Schottky, symbol Device:D_Schottky
- added Q1: AO3401A, Package_TO_SOT_SMD:SOT-23, symbol Transistor_FET:AO3401A
- added Q2: LBSS84LT1G, symbol Device:Q_PMOS_SDG
- added R1, R6: 0, symbol Device:R_Small
- added R5: 10k, symbol Device:R_Small
- added U2: XC6206PxxxMR, Package_TO_SOT_SMD:SOT-23-3, symbol Regulator_Linear:XC6206PxxxMR
- added U3: OP07, symbol Amplifier_Operational:OP07
- renumbered R1 to R2, R2 to R3, R3 to R4
Connections:
- net 3V3: now also C4.1, C5.1, U2.2 (VO)
- net GND: now also C3.2, C4.2, C5.2, Q2.3 (G), R5.1, U2.1 (GND), U3.2 (-), U3.4 (V-)
- net USB_IN_5V: now also R1.1; no longer C1.2, LED1.2 (A), LED2.2 (A), U1.4 (VCC), U1.8 (CE)
- net V_BAT+: now also Q1.2 (S), R6.1; no longer C2.1, U1.5 (BAT)
- new net: C1.2, D1.2 (A), LED1.2 (A), LED2.2 (A), Q1.1 (G), R1.2, R5.2, U1.4 (VCC), U1.8 (CE)
- new net: C2.1, R6.2, U1.5 (BAT)
- new net: D2.1 (K), Q2.1 (S)
- new net: Q2.2 (D), U3.3 (+)
- new net CHRG_OUT: D1.1 (K), D2.2 (A), Q1.3 (D), U3.7 (V+)
- new net UVLO_3V3: C3.1, U2.3 (VI), U3.6
- no-connect marks 0 -> 2
Other:
- note added: "Section B: 3V3 Regulator"
- note added: "Section C: UVLO and Polarity Protection"
- note removed: "Section B: Voltage Regulator"
- company: (none) -> Group 3
- title: (none) -> Power Subsystem
- moved on the sheet: BT1, C1, C2, LED1, LED2, R2, R3, R4, U1
