File: PCB/microcontroller_interfacing.kicad_sch (KiCad schematic)
At the start: 25 parts, among them J12 Conn_01x01, U6 CH340C

Commit message: Add GPIO pins and crystal oscillator
Parts:
- added C16, C17: 10pF, symbol Device:C_Small
- added Y1: 8MHz Crystal, symbol Device:Crystal
Connections:
- net GND: now also C16.2, C17.2
- net USB 5V: now also J?.13 (Pin_13), J?.13 (Pin_13)
- net OSC IN: now reaches J?.11 (Pin_11), J?.11 (Pin_11)
- net OSC IN: now also C17.1, Y1.2
- net OSC OUT: now reaches J?.12 (Pin_12), J?.12 (Pin_12)
- net OSC OUT: now also C16.1, Y1.1
- net GPIO 1: now reaches J?.12 (Pin_12), J?.12 (Pin_12)
Other:
- note added: "An external crytal oscillator that generates a 8MHz clock frequency"
- note added: "Clock Generator"
- moved on the sheet: R36
