File: PCB/microcontroller_interfacing.kicad_sch (KiCad schematic)
At the start: 28 parts, among them J7 Conn_01x01_Pin, U7 CH340C, Y1 C252310

Commit message: PCB_Design_1
Parts:
- J? (x2): footprint Connector_PinSocket_2.54mm:PinSocket_1x24_P2.54mm_Vertical -> Connector_PinHeader_2.54mm:PinHeader_1x24_P2.54mm_Vertical
Connections:
- net USB 5V: no longer J?.13 (Pin_13), J?.13 (Pin_13)
- new net: J?.13 (Pin_13), J?.13 (Pin_13)
Changed lines of the file:
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@@
-    (effects (font (size 1.27 1.27)) (justify left))
-  )
-  (hierarchical_label "USB 5V" (shape input) (at 193.04 67.31 0) (fields_autoplaced)
     (effects (font (size 1.27 1.27)) (justify left))
   )
@@
       (effects (font (size 1.27 1.27)) (justify right))
     )
-    (property "Footprint" "Connector_PinSocket_2.54mm:PinSocket_1x24_P2.54mm_Vertical" (at 264.795 67.31 0)
+    (property "Footprint" "Connector_PinHeader_2.54mm:PinHeader_1x24_P2.54mm_Vertical" (at 264.795 67.31 0)
       (effects (font (size 1.27 1.27)) hide)
     )
@@
       (effects (font (size 1.27 1.27)) (justify right))
     )
-    (property "Footprint" "Connector_PinSocket_2.54mm:PinSocket_1x24_P2.54mm_Vertical" (at 186.055 64.77 0)
-      (effects (font (size 1.27 1.27)) hide)
-    )
+    (property "Footprint" "Connector_PinHeader_2.54mm:PinHeader_1x24_P2.54mm_Vertical" (at 186.055 64.77 0)
+      (effects (font (size 1.27 1.27)) hide)
+    )

Commit message: fixing of PCB Design
Connections:
- net USART_RX: no longer J?.7 (Pin_7), J?.7 (Pin_7)
- net USART_TX: no longer J?.6 (Pin_6), J?.6 (Pin_6)
- new net: J?.6 (Pin_6), J?.6 (Pin_6)
- new net: J?.7 (Pin_7), J?.7 (Pin_7)
- no-connect marks 11 -> 12
Changed lines of the file:
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@@
   (no_connect (at 139.7 111.76))
   (no_connect (at 139.7 121.92))
+  (no_connect (at 119.38 106.68))
   (no_connect (at 57.15 85.09))
   (no_connect (at 139.7 116.84))
@@
     )
   )
-  (global_label "USART_RX" (shape input) (at 246.38 80.01 0) (fields_autoplaced)
-    (effects (font (size 1.27 1.27)) (justify left))
-    (property "Intersheetrefs" "${INTERSHEET_REFS}" (at 258.5991 80.01 0)
-      (effects (font (size 1.27 1.27)) (justify left) hide)
-    )
-  )
   (global_label "USB D+" (shape input) (at 151.13 38.1 0) (fields_autoplaced)
     (effects (font (size 1.27 1.27)) (justify left))
@@
       (effects (font (size 1.27 1.27)) (justify left) hide)
     )
-  )
-  (global_label "USART_TX" (shape input) (at 246.38 82.55 0) (fields_autoplaced)
-    (effects (font (size 1.27 1.27)) (justify left))
-    (property "Intersheetrefs" "${INTERSHEET_REFS}" (at 258.2967 82.55 0)
-      (effects (font (size 1.27 1.27)) (justify left) hide)
-    )

Commit message: Pins not Sockets
Parts:
- J7: footprint Connector_PinSocket_2.54mm:PinSocket_1x01_P2.54mm_Vertical -> Connector_PinHeader_2.54mm:PinHeader_1x01_P2.54mm_Vertical
- J?: footprint Connector_PinSocket_2.54mm:PinSocket_1x10_P2.54mm_Vertical -> Connector_PinHeader_2.54mm:PinHeader_1x10_P2.54mm_Vertical
Changed lines of the file:
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@@
       (effects (font (size 1.27 1.27)))
     )
-    (property "Footprint" "Connector_PinSocket_2.54mm:PinSocket_1x10_P2.54mm_Vertical" (at 54.61 80.01 0)
+    (property "Footprint" "Connector_PinHeader_2.54mm:PinHeader_1x10_P2.54mm_Vertical" (at 54.61 80.01 0)
       (effects (font (size 1.27 1.27)) hide)
     )
@@
       (effects (font (size 1.27 1.27)) (justify left))
     )
-    (property "Footprint" "Connector_PinSocket_2.54mm:PinSocket_1x01_P2.54mm_Vertical" (at 179.07 127 0)
-      (effects (font (size 1.27 1.27)) hide)
-    )
+    (property "Footprint" "Connector_PinHeader_2.54mm:PinHeader_1x01_P2.54mm_Vertical" (at 179.07 127 0)
+      (effects (font (size 1.27 1.27)) hide)
+    )
