File: PCB/Sensor_Module.kicad_sch (KiCad schematic)
At the start: 16 parts, among them J2 Conn_01x01_Pin, J5 Conn_01x02_Pin, U7 VL6180

Commit message: commenting of trace thicknesses
Parts:
- renumbered J2 to J3, J5 to J4, U7 to U4
Changed lines of the file:
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@@
       (project "HAT"
         (path "/40f36b19-a08c-43e7-88a6-ec8387939712/2460aa4e-e7b3-4d03-ad75-cceb37813eec"
-          (reference "#PWR024") (unit 1)
+          (reference "#PWR023") (unit 1)
         )
       )
@@
       (project "HAT"
         (path "/40f36b19-a08c-43e7-88a6-ec8387939712/2460aa4e-e7b3-4d03-ad75-cceb37813eec"
-          (reference "R7") (unit 1)
+          (reference "R17") (unit 1)
         )
       )
@@
       (project "HAT"
         (path "/40f36b19-a08c-43e7-88a6-ec8387939712/2460aa4e-e7b3-4d03-ad75-cceb37813eec"
-          (reference "R27") (unit 1)
+          (reference "R23") (unit 1)
         )
       )
@@
       (project "HAT"
         (path "/40f36b19-a08c-43e7-88a6-ec8387939712/2460aa4e-e7b3-4d03-ad75-cceb37813eec"
-          (reference "C8") (unit 1)
+          (reference "C6") (unit 1)
         )
       )
@@
   (symbol (lib_id "Connector:Conn_01x02_Pin") (at 171.45 81.28 0) (unit 1)
     (in_bom yes) (on_board yes) (dnp no)
-    (property "Reference" "J5" (at 171.45 78.74 0)
+    (property "Reference" "J4" (at 171.45 78.74 0)
       (effects (font (size 1.27 1.27)))
     )
@@
       (project "HAT"
         (path "/40f36b19-a08c-43e7-88a6-ec8387939712/2460aa4e-e7b3-4d03-ad75-cceb37813eec"
-          (reference "J5") (unit 1)
+          (reference "J4") (unit 1)
         )
       )
@@
       (project "HAT"
         (path "/40f36b19-a08c-43e7-88a6-ec8387939712/2460aa4e-e7b3-4d03-ad75-cceb37813eec"
-          (reference "#PWR021") (unit 1)
+          (reference "#PWR018") (unit 1)
         )
       )
@@
       (project "HAT"
         (path "/40f36b19-a08c-43e7-88a6-ec8387939712/2460aa4e-e7b3-4d03-ad75-cceb37813eec"
-          (reference "#PWR019") (unit 1)
+          (reference "#PWR021") (unit 1)
         )
       )
@@
       (project "HAT"
         (path "/40f36b19-a08c-43e7-88a6-ec8387939712/2460aa4e-e7b3-4d03-ad75-cceb37813eec"
-          (reference "C9") (unit 1)
+          (reference "C7") (unit 1)
         )
       )
@@
       (project "HAT"
         (path "/40f36b19-a08c-43e7-88a6-ec8387939712/2460aa4e-e7b3-4d03-ad75-cceb37813eec"
-          (reference "R25") (unit 1)
+          (reference "R21") (unit 1)
         )
       )
@@
       (project "HAT"
         (path "/40f36b19-a08c-43e7-88a6-ec8387939712/2460aa4e-e7b3-4d03-ad75-cceb37813eec"
-          (reference "R11") (unit 1)
+          (reference "R19") (unit 1)
         )
       )
@@
       (project "HAT"
         (path "/40f36b19-a08c-43e7-88a6-ec8387939712/2460aa4e-e7b3-4d03-ad75-cceb37813eec"
-          (reference "C6") (unit 1)
+          (reference "C8") (unit 1)
         )
       )
@@
   (symbol (lib_id "Proximity Sensor:VL6180") (at 60.96 45.72 0) (mirror y) (unit 1)
     (in_bom yes) (on_board yes) (dnp no)
-    (property "Reference" "U7" (at 60.96 31.75 0)
+    (property "Reference" "U4" (at 60.96 31.75 0)
       (effects (font (size 1.27 1.27)))
     )
@@
       (project "HAT"
         (path "/40f36b19-a08c-43e7-88a6-ec8387939712/2460aa4e-e7b3-4d03-ad75-cceb37813eec"
-          (reference "U7") (unit 1)
+          (reference "U4") (unit 1)
         )
       )
@@
       (project "HAT"
         (path "/40f36b19-a08c-43e7-88a6-ec8387939712/2460aa4e-e7b3-4d03-ad75-cceb37813eec"
-          (reference "C7") (unit 1)
+          (reference "C9") (unit 1)
         )
       )
@@
       (project "HAT"
         (path "/40f36b19-a08c-43e7-88a6-ec8387939712/2460aa4e-e7b3-4d03-ad75-cceb37813eec"
-          (reference "#PWR018") (unit 1)
+          (reference "#PWR020") (unit 1)
         )
       )
@@
       (project "HAT"
         (path "/40f36b19-a08c-43e7-88a6-ec8387939712/2460aa4e-e7b3-4d03-ad75-cceb37813eec"
-          (reference "R14") (unit 1)
+          (reference "R20") (unit 1)
         )
       )
@@
       (project "HAT"
         (path "/40f36b19-a08c-43e7-88a6-ec8387939712/2460aa4e-e7b3-4d03-ad75-cceb37813eec"
-          (reference "U4") (unit 1)
+          (reference "U5") (unit 1)
         )
       )
@@
       (project "HAT"
         (path "/40f36b19-a08c-43e7-88a6-ec8387939712/2460aa4e-e7b3-4d03-ad75-cceb37813eec"
-          (reference "R28") (unit 1)
+          (reference "R24") (unit 1)
         )
       )
@@
       (project "HAT"
         (path "/40f36b19-a08c-43e7-88a6-ec8387939712/2460aa4e-e7b3-4d03-ad75-cceb37813eec"
-          (reference "R26") (unit 1)
+          (reference "R22") (unit 1)
         )
       )
@@
   (symbol (lib_id "Connector:Conn_01x01_Pin") (at 105.41 95.25 270) (unit 1)
     (in_bom yes) (on_board yes) (dnp no) (fields_autoplaced)
-    (property "Reference" "J2" (at 106.68 95.25 90)
+    (property "Reference" "J3" (at 106.68 95.25 90)
       (effects (font (size 1.27 1.27)) (justify left))
     )
@@
       (project "HAT"
         (path "/40f36b19-a08c-43e7-88a6-ec8387939712/2460aa4e-e7b3-4d03-ad75-cceb37813eec"
-          (reference "J2") (unit 1)
+          (reference "J3") (unit 1)
         )
       )
@@
       (project "HAT"
         (path "/40f36b19-a08c-43e7-88a6-ec8387939712/2460aa4e-e7b3-4d03-ad75-cceb37813eec"
-          (reference "#PWR017") (unit 1)
+          (reference "#PWR019") (unit 1)
         )
       )
@@
       (project "HAT"
         (path "/40f36b19-a08c-43e7-88a6-ec8387939712/2460aa4e-e7b3-4d03-ad75-cceb37813eec"
-          (reference "R10") (unit 1)
-        )
-      )
+          (reference "R18") (unit 1)
+        )
+      )
