File: PCB/Logic_Level_Shifting.kicad_sch (KiCad schematic)
At the start: 24 parts, among them Q4 BSS138, Q5 BSS138, Q6 BSS138, Q7 BSS138

Commit message: literally all the footprints
Parts:
- J? (x4): footprint (none) -> Connector_PinSocket_2.54mm:PinSocket_1x02_P2.54mm_Vertical
- Q4, Q5, Q6, Q7: footprint Package_TO_SOT_SMD:SOT-23 -> JLC_Mosfet:SOT-23-3_L2.9-W1.3-P1.90-LS2.4-BR
- R? (x16): footprint (none) -> Resistor_SMD:R_0805_2012Metric

Commit message: PCB_Design_1
Parts:
- J? (x4): footprint Connector_PinSocket_2.54mm:PinSocket_1x02_P2.54mm_Vertical -> Connector_PinHeader_2.54mm:PinHeader_1x02_P2.54mm_Vertical
Changed lines of the file:
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@@
       (effects (font (size 1.27 1.27)) (justify right) hide)
     )
-    (property "Footprint" "Connector_PinSocket_2.54mm:PinSocket_1x02_P2.54mm_Vertical" (at 82.55 148.59 0)
+    (property "Footprint" "Connector_PinHeader_2.54mm:PinHeader_1x02_P2.54mm_Vertical" (at 82.55 148.59 0)
       (effects (font (size 1.27 1.27)) hide)
     )
@@
       (effects (font (size 1.27 1.27)) (justify right) hide)
     )
-    (property "Footprint" "Connector_PinSocket_2.54mm:PinSocket_1x02_P2.54mm_Vertical" (at 189.23 68.58 0)
+    (property "Footprint" "Connector_PinHeader_2.54mm:PinHeader_1x02_P2.54mm_Vertical" (at 189.23 68.58 0)
       (effects (font (size 1.27 1.27)) hide)
     )
@@
       (effects (font (size 1.27 1.27)) (justify right) hide)
     )
-    (property "Footprint" "Connector_PinSocket_2.54mm:PinSocket_1x02_P2.54mm_Vertical" (at 83.82 68.58 0)
+    (property "Footprint" "Connector_PinHeader_2.54mm:PinHeader_1x02_P2.54mm_Vertical" (at 83.82 68.58 0)
       (effects (font (size 1.27 1.27)) hide)
     )
@@
       (effects (font (size 1.27 1.27)) (justify right) hide)
     )
-    (property "Footprint" "Connector_PinSocket_2.54mm:PinSocket_1x02_P2.54mm_Vertical" (at 195.58 148.59 0)
-      (effects (font (size 1.27 1.27)) hide)
-    )
+    (property "Footprint" "Connector_PinHeader_2.54mm:PinHeader_1x02_P2.54mm_Vertical" (at 195.58 148.59 0)
+      (effects (font (size 1.27 1.27)) hide)
+    )

Commit message: sensor layout pcb
Changed lines of the file:
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@@
     (in_bom yes) (on_board yes) (dnp no) (fields_autoplaced)
     (property "Reference" "R?" (at 63.5 48.26 90)
-      (effects (font (size 1.27 1.27)) hide)
+      (effects (font (size 1.27 1.27)))
     )
     (property "Value" "0" (at 63.5 50.8 90)
@@
     (in_bom yes) (on_board yes) (dnp no) (fields_autoplaced)
     (property "Reference" "R?" (at 62.23 128.27 90)
-      (effects (font (size 1.27 1.27)) hide)
+      (effects (font (size 1.27 1.27)))
     )
     (property "Value" "0" (at 62.23 130.81 90)
@@
     (in_bom yes) (on_board yes) (dnp no) (fields_autoplaced)
     (property "Reference" "R?" (at 175.26 128.27 90)
-      (effects (font (size 1.27 1.27)) hide)
+      (effects (font (size 1.27 1.27)))
     )
     (property "Value" "0" (at 175.26 130.81 90)
@@
     (in_bom yes) (on_board yes) (dnp no) (fields_autoplaced)
     (property "Reference" "R?" (at 168.91 48.26 90)
-      (effects (font (size 1.27 1.27)) hide)
+      (effects (font (size 1.27 1.27)))
     )
     (property "Value" "0" (at 168.91 50.8 90)
